File: OpenFlex_SMD/mcu.kicad_sch (KiCad schematic)
At the start: 1 part

Commit message: Updated BOM
Parts:
- removed A1: Arduino_Nano_Every, Module:Arduino_Nano_WithMountingHoles, symbol MCU_Module:Arduino_Nano_Every
- added U2: ESP32-S3-WROOM-1, RF_Module:ESP32-S3-WROOM-1, symbol RF_Module:ESP32-S3-WROOM-1
Connections:
- net GND: now also U2.1 (GND), U2.40 (GND), U2.41 (GND)
