File: EmulatorBoard/EmulatorBoard.kicad_sch (KiCad schematic)
At the start: 21 parts, among them J1 Conn_02x04_Odd_Even, J2 Screw_Terminal_01x10, Q1 BC338, Q2 IRF740, Q3 IRF740, Q4 IRF740, Q5 IRF740, Q6 BC338, U1 TC4424, U2 TC4424

Commit message: Updated and sourced EmulatoBoard (DevBoard)
Parts:
- removed J1: Conn_02x04_Odd_Even, Connector_PinHeader_2.54mm:PinHeader_2x04_P2.54mm_Vertical, symbol Connector_Generic:Conn_02x04_Odd_Even
- removed Q1, Q6: BC338, Package_TO_SOT_THT:TO-92_Inline, symbol Transistor_BJT:BC338
- removed Q2, Q3, Q4, Q5: IRF740, Package_TO_SOT_THT:TO-220-3_Horizontal_TabDown, symbol Transistor_FET:IRF740
- removed RV1: 100k Lin, Potentiometer_THT:Potentiometer_Omeg_PC16BU_Horizontal, symbol Device:R_Potentiometer
- removed U1, U2: TC4424, Package_DIP:DIP-8_W7.62mm_Socket, symbol IC_Automotive:TC4424
- added C1, C3: 10uF, Capacitor_THT:CP_Radial_D5.0mm_P2.00mm, symbol Device:C_Polarized
- added C2, C4: 1nF, Capacitor_THT:C_Disc_D5.0mm_W2.5mm_P2.50mm, symbol Device:C
- added C5: 100nF, Capacitor_THT:C_Disc_D5.0mm_W2.5mm_P2.50mm, symbol Device:C
- added J1: Screw_Terminal_01x02, TerminalBlock_Phoenix:TerminalBlock_Phoenix_MKDS-1,5-2-5.08_1x02_P5.08mm_Horizontal, symbol Connector:Screw_Terminal_01x02
- added JP1: SolderJumper_2_Open, Jumper:SolderJumper-2_P1.3mm_Open_RoundedPad1.0x1.5mm, symbol Jumper:SolderJumper_2_Open
- added Q1, Q2, Q3, Q4, Q5, Q6: 2N2222A, Package_TO_SOT_THT:TO-92L_Inline_Wide, symbol Transistor_BJT:Q_NPN_CBE
- added R1, R5, R7, R8: 1k, Resistor_THT:R_Axial_DIN0207_L6.3mm_D2.5mm_P10.16mm_Horizontal, symbol Device:R
- added RV4: 100k Lin, OpenFlex_FootPrint_Lib:PTN091V100115K1B, symbol Device:R_Potentiometer
- added U1: LM7805_TO220, Package_TO_SOT_THT:TO-220-3_Vertical, symbol Regulator_Linear:LM7805_TO220
- C6: renamed from C1; footprint Capacitor_THT:C_Disc_D7.5mm_W5.0mm_P7.50mm -> Capacitor_THT:C_Rect_L7.2mm_W6.0mm_P5.00mm; Manufacturer_Name (none) -> KEMET; Manufacturer_Part_Number (none) -> R82EC4100SH70J; Mouser_Part_Number (none) -> 80-R82EC4100SH70J; URL (none) -> https://www.mouser.fr/ProductDetail/KEMET/R82EC4100SH70J?qs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
- C7: renamed from C2; footprint Capacitor_THT:C_Disc_D7.5mm_W5.0mm_P7.50mm -> Capacitor_THT:C_Rect_L7.2mm_W4.5mm_P5.00mm_FKS2_FKP2_MKS2_MKP2; Manufacturer_Name (none) -> KEMET; Manufacturer_Part_Number (none) -> 82IC3100Z360J; Mouser_Part_Number (none) -> 80-R82IC3100Z360J; URL (none) -> https://www.mouser.fr/ProductDetail/KEMET/R82IC3100Z360J?qs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
- J2: Manufacturer_Name (none) -> Phoenix Contact; Manufacturer_Part_Number (none) -> 1727094; Mouser_Part_Number (none) -> 651-1727094; URL (none) -> https://www.mouser.fr/ProductDetail/Phoenix-Contact/1727094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
- R2, R3, R4: Manufacturer_Name (none) -> YAGEO; Manufacturer_Part_Number (none) -> MFR-25FBF52-1K; Mouser_Part_Number (none) -> 603-MFR-25FBF52-1K; URL (none) -> https://www.mouser.fr/ProductDetail/YAGEO/MFR-25FBF52-1K?qs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
- R6: renamed from R1; Manufacturer_Name (none) -> YAGEO; Manufacturer_Part_Number (none) -> MFR-25FBF52-1K; Mouser_Part_Number (none) -> 603-MFR-25FBF52-1K; URL (none) -> https://www.mouser.fr/ProductDetail/YAGEO/MFR-25FBF52-1K?qs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
- RV1: renamed from RV4; footprint Potentiometer_THT:Potentiometer_Omeg_PC16BU_Horizontal -> OpenFlex_FootPrint_Lib:PTN091V100115K1B; Manufacturer_Name (none) -> Same Sky; Manufacturer_Part_Number (none) -> PTN091V100115K1B; Mouser_Part_Number (none) -> 179-PTN091V100115K1B; URL (none) -> https://www.mouser.fr/ProductDetail/Same-Sky/PTN091-V100115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
- RV2, RV3: footprint Potentiometer_THT:Potentiometer_Omeg_PC16BU_Horizontal -> OpenFlex_FootPrint_Lib:PTN091V100115K1B; Manufacturer_Name (none) -> Same Sky; Manufacturer_Part_Number (none) -> PTN091V100115K1B; Mouser_Part_Number (none) -> 179-PTN091V100115K1B; URL (none) -> https://www.mouser.fr/ProductDetail/Same-Sky/PTN091-V100115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
Connections:
- net +12V: now also J2.9 (Pin_9), C1.1, C2.1, J1.1 (Pin_1), U1.1 (VI); no longer J2.2 (Pin_2)
- net FREQ_Pot: now also RV1.2
- net Flex_SNSR_Signal: now also J2.3 (Pin_3), Q6.3 (E), R8.2; no longer J2.8 (Pin_8), R2.2
- net GD_CH1: now also R1.1
- net GD_CH2: now also R3.1
- net GD_CH3: now also R2.1
- net GD_CH4: now also R4.1
- net GND: now also J2.10 (Pin_10), C1.2, C2.2, C3.2, C4.2, C5.2, J1.2 (Pin_2), Q1.3 (E), Q2.3 (E), Q3.3 (E), Q4.3 (E), Q5.3 (E), R8.1, RV4.3, U1.2 (GND); no longer J2.1 (Pin_1), R2.1
- net INJ_CH1: now also J2.8 (Pin_8), Q1.1 (C); no longer J2.3 (Pin_3)
- net INJ_CH2: now also J2.7 (Pin_7), Q3.1 (C); no longer J2.4 (Pin_4)
- net INJ_CH3: now also J2.6 (Pin_6), Q2.1 (C); no longer J2.5 (Pin_5)
- net INJ_CH4: now also J2.5 (Pin_5), Q4.1 (C); no longer J2.6 (Pin_6)
- net MCU_D3: now also R5.1; no longer R3.1
- net Temp_+: now also J2.2 (Pin_2), R7.2; no longer J2.9 (Pin_9), R4.2
- net Temp_-: now also J2.1 (Pin_1), Q5.1 (C), R7.1; no longer J2.10 (Pin_10), R4.1
- net Temp_Pot: now also RV4.2; no longer RV1.2
- net VDD: now also A1.5V, C3.1, C4.1, C5.1, JP1.1 (A), Q6.1 (C), U1.3 (VO)
- net at R6.2: now also Q6.2 (B)
- net at C7.1: now also Q5.2 (B), R5.2; no longer R3.2
- net +5V renamed AREF_Pin
- net AREF_Pin: now also JP1.2 (B), RV4.1; no longer A1.5V
- new net: Q2.2 (B), R2.2
- new net: Q1.2 (B), R1.2
- new net: Q4.2 (B), R4.2
- new net: Q3.2 (B), R3.2
Other:
- note added: "Injector Drive _ ECU Equivalent"
- note removed: "Todo : Ajouter Aref correctement"
- moved on the sheet: C6, C7, J2, R6, RV1

Commit message: Updated BOM
Other:
- removed sheet Power
Changed lines of the file:
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@@
-		)
-	)
-	(sheet
-		(at 152.4 177.8)
-		(size 12.7 12.7)
-		(exclude_from_sim no)
-		(in_bom yes)
-		(on_board yes)
-		(dnp no)
-		(fields_autoplaced yes)
-		(stroke
-			(width 0.1524)
-			(type solid)
-		)
-		(fill
-			(color 0 0 0 0)
-		)
-		(property "Sheetname" "Power"
-			(at 152.4 177.0884 0)
-			(show_name no)
-			(do_not_autoplace no)
-			(effects
-				(font
-					(size 1.27 1.27)
-				)
-				(justify left bottom)
-			)
-		)
-		(property "Sheetfile" "pwr.kicad_sch"
-			(at 152.4 191.0846 0)
-			(show_name no)
-			(do_not_autoplace no)
-			(effects
-				(font
-					(size 1.27 1.27)
-				)
-				(justify left top)
-			)
-		)
-		(instances
-			(project "EmulatorBoard"
-				(path "/f1104bbf-8d85-4011-a1d1-ffdecdb41ac7"
-					(page "2")
-				)
-			)
 		)
 	)
