File: OpenFlex_Prototype/OpenFlex_Proto_THT.kicad_pcb (KiCad board)
At the start: 2 copper layers, 107.8 x 69.9 mm, 43 parts, among them J2 Molex MAX150_2x10, M3 MountingHole_3.2mm_M3_DIN965_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, Q1 IRF740, Q2 IRF740, Q3 IRF740, Q4 IRF740, U1 ESP32-S2-DEVKITC-1, U2 LM324, U3 TC4424, U4 TC4424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

Commit message: Updated BOM
Parts:
- Q1, Q2, Q3, Q4: value IRF740 -> STP80NF55-08
- moved R3 3.20 mm to (181.6, 94.5)
- moved R4 3.20 mm to (184.8, 94.5)
- moved U1 0.40 mm to (242.5, 83.2)
- moved Q2 0.06 mm to (194.7, 89.7)
Routing:
- net VDD: track 17.3 -> 127.0 mm, vias 0 -> 1
- net /Connector/INJ_CH4: track 25.7 -> 34.0 mm
- net VSS: track 92.9 -> 92.2 mm
- net /IO_Drivers/Temp_Signal: track 120.6 -> 121.3 mm
- net GND: vias 174 -> 187

Commit message: Updated BOM
Parts:
- turned C2 to 90 degrees
